File: led_module.kicad_sch (KiCad schematic)
At the start: 0 parts

Commit message: add libraries and add components in schematic
Parts:
- added D1, D2, D3, D4, D5, D6, D7, D8: GREEN, symbol 0_Led:LED
- added J1: Conn_01x10, symbol 0_Connector_Generic:Conn_01x10
- added R1, R2, R3, R4, R5, R6, R7, R8: 330, symbol 0_Resistor:R
Connections:
- new net +5V: J1.10 (Pin_10)
- new net C-R1: J1.2 (Pin_2), R1.1
- new net C-R2: J1.3 (Pin_3), R2.1
- new net C-R3: J1.4 (Pin_4), R3.1
- new net C-R4: J1.5 (Pin_5), R4.1
- new net C-R5: J1.6 (Pin_6), R5.1
- new net C-R6: J1.7 (Pin_7), R6.1
- new net C-R7: J1.8 (Pin_8), R7.1
- new net C-R8: J1.9 (Pin_9), R8.1
- new net GND: D1.1 (K), D2.1 (K), D3.1 (K), D4.1 (K), D5.1 (K), D6.1 (K), D7.1 (K), D8.1 (K), J1.1 (Pin_1)
- new net R-L1: D1.2 (A), R1.2
- new net R-L2: D2.2 (A), R2.2
- new net R-L3: D3.2 (A), R3.2
- new net R-L4: D4.2 (A), R4.2
- new net R-L5: D5.2 (A), R5.2
- new net R-L6: D6.2 (A), R6.2
- new net R-L7: D7.2 (A), R7.2
- new net R-L8: D8.2 (A), R8.2
Other:
- company: (none) -> Magz Industry
- title: (none) -> LED MODULE

Commit message: create footprint libraries and add footprint in componets
Parts:
- D1, D2, D3, D4, D5, D6, D7, D8: footprint (none) -> 0_Led:LED_0805_2012Metric
- J1: footprint (none) -> 0_Connector_Generic:PinHeader_1x10_P2.54mm_Vertical
- R1, R2, R3, R4, R5, R6, R7, R8: footprint (none) -> 0_Resistor:R_0805_2012Metric
Changed lines of the file:
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@@
 			)
 		)
-		(property "Footprint" ""
+		(property "Footprint" "0_Resistor:R_0805_2012Metric"
 			(at 170.942 81.28 90)
 			(effects
@@
 			)
 		)
-		(property "Footprint" ""
+		(property "Footprint" "0_Resistor:R_0805_2012Metric"
 			(at 132.842 81.28 90)
 			(effects
@@
 			)
 		)
-		(property "Footprint" ""
+		(property "Footprint" "0_Led:LED_0805_2012Metric"
 			(at 96.52 100.33 0)
 			(effects
@@
 			)
 		)
-		(property "Footprint" ""
+		(property "Footprint" "0_Led:LED_0805_2012Metric"
 			(at 160.02 100.33 0)
 			(effects
@@
 			)
 		)
-		(property "Footprint" ""
+		(property "Footprint" "0_Resistor:R_0805_2012Metric"
 			(at 82.042 81.28 90)
 			(effects
@@
 			)
 		)
-		(property "Footprint" ""
+		(property "Footprint" "0_Led:LED_0805_2012Metric"
 			(at 147.32 100.33 0)
 			(effects
@@
 			)
 		)
-		(property "Footprint" ""
+		(property "Footprint" "0_Led:LED_0805_2012Metric"
 			(at 121.92 100.33 0)
 			(effects
@@
 			)
 		)
-		(property "Footprint" ""
+		(property "Footprint" "0_Resistor:R_0805_2012Metric"
 			(at 158.242 81.28 90)
 			(effects
@@
 			)
 		)
-		(property "Footprint" ""
+		(property "Footprint" "0_Led:LED_0805_2012Metric"
 			(at 172.72 100.33 0)
 			(effects
@@
 			)
 		)
-		(property "Footprint" ""
+		(property "Footprint" "0_Led:LED_0805_2012Metric"
 			(at 83.82 100.33 0)
 			(effects
@@
 			)
 		)
-		(property "Footprint" ""
+		(property "Footprint" "0_Led:LED_0805_2012Metric"
 			(at 109.22 100.33 0)
 			(effects
@@
 			)
 		)
-		(property "Footprint" ""
+		(property "Footprint" "0_Connector_Generic:PinHeader_1x10_P2.54mm_Vertical"
 			(at 46.99 67.31 0)
 			(effects
@@
 			)
 		)
-		(property "Footprint" ""
+		(property "Footprint" "0_Resistor:R_0805_2012Metric"
 			(at 120.142 81.28 90)
 			(effects
@@
 			)
 		)
-		(property "Footprint" ""
+		(property "Footprint" "0_Resistor:R_0805_2012Metric"
 			(at 94.742 81.28 90)
 			(effects
@@
 			)
 		)
-		(property "Footprint" ""
+		(property "Footprint" "0_Led:LED_0805_2012Metric"
 			(at 134.62 100.33 0)
 			(effects
@@
 			)
 		)
-		(property "Footprint" ""
+		(property "Footprint" "0_Resistor:R_0805_2012Metric"
 			(at 107.442 81.28 90)
 			(effects
@@
 			)
 		)
-		(property "Footprint" ""
+		(property "Footprint" "0_Resistor:R_0805_2012Metric"
 			(at 145.542 81.28 90)
 			(effects
